Commit message: revise

File: src/jaka_a5_description/urdf/jaka_a5.urdf (robot description, URDF)
Before this commit: robot jaka_a5, 8 links, 7 joints
Links:
- link J1: geometry collision mesh filename=package://jaka_a5_description/meshes/jaka_a5_meshes/J1.STL; visual mesh filename=package://jaka_a5_description/meshes/jaka_a5_meshes/J1.STL
- link J2: geometry collision mesh filename=package://jaka_a5_description/meshes/jaka_a5_meshes/J2.STL; visual mesh filename=package://jaka_a5_description/meshes/jaka_a5_meshes/J2.STL
- link J3: geometry collision mesh filename=package://jaka_a5_description/meshes/jaka_a5_meshes/J3.STL; visual mesh filename=package://jaka_a5_description/meshes/jaka_a5_meshes/J3.STL
- link J4: geometry collision mesh filename=package://jaka_a5_description/meshes/jaka_a5_meshes/J4.STL; visual mesh filename=package://jaka_a5_description/meshes/jaka_a5_meshes/J4.STL
- link J5: geometry collision mesh filename=package://jaka_a5_description/meshes/jaka_a5_meshes/J5.STL; visual mesh filename=package://jaka_a5_description/meshes/jaka_a5_meshes/J5.STL
- link J6: geometry collision mesh filename=package://jaka_a5_description/meshes/jaka_a5_meshes/J6.STL; visual mesh filename=package://jaka_a5_description/meshes/jaka_a5_meshes/J6.STL
- link base_link: geometry collision mesh filename=package://jaka_a5_description/meshes/jaka_a5_meshes/base_li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; visual mesh filename=package://jaka_a5_description/meshes/jaka_a5_meshes/base_li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
